File: Schematy eagle/Falownik/falownik.sch (EAGLE design)
At the start: 16 parts, among them Q1 BSS101, Q2 BSS101, Q3 BSS101, Q4 BSS101, Q5 BSS101, Q6 BSS101, X1 87758-0216, X2 87758-0216, X3 87758-0216, X4 87758-0216

Commit message: Falownik update
Parts:
- added U$1, U$10, U$11, U$12, U$13, U$14, U$15, U$16, U$17, U$18, U$2, U$3, U$4, U$5, U$6, U$7, U$8, U$9: CURRENT_MEAS_D_V02, current_meas:CURRENT_MEAS_D_V02
- added X10, X11, X12, X13, X5, X6, X7, X8, X9: 87758-0216, con-molex:87758-0216
Connections:
- new net GND: D2.A, D4.A, D6.A, Q2.S, Q4.S, Q6.S, U$1.GND, U$10.GND, U$11.GND, U$12.GND, U$13.GND, U$14.GND, U$15.GND, U$16.GND, U$17.GND, U$18.GND, U$2.GND, U$3.GND, U$4.GND, U$5.GND, U$6.GND, U$7.GND, U$8.GND, U$9.GND, X1-2.S
- new net L4: D3.A, Q3.S, U$7.OUT
- new net L5: Q4.D, U$11.IN, U$7.IN
- new net L6: Q3.D, U$12.IN, U$8.IN
- new net L7: D5.A, Q5.S, U$13.OUT
- new net L8: Q6.D, U$13.IN, U$17.IN
- new net L9: Q5.D, U$14.IN, U$18.IN
- new net N$1: D1.C, U$6.OUT
- new net N$10: D5.C, U$18.OUT
- new net N$4: D4.C, U$11.OUT
- new net N$5: D2.C, U$5.OUT
- new net N$6: D3.C, U$12.OUT
- new net N$9: D6.C, U$17.OUT
- new net VCC: U$14.OUT, U$2.OUT, U$8.OUT, X1-1.S
- new net VCC1: Q3.G, U$9.OUT
- new net VCC2: Q4.G, U$10.OUT
- new net VCC3: Q5.G, U$15.OUT
- new net VCC4: Q6.G, U$16.OUT
- new net VCC5: Q1.G, U$3.OUT
- new net VCC6: Q2.G, U$4.OUT
- new net V_D11: U$6.VO, X11-1.S
- new net V_D12: U$12.VO, X12-1.S
- new net V_D13: U$18.VO, X13-1.S
- new net V_D21: U$5.VO, X11-2.S
- new net V_D22: U$11.VO, X12-2.S
- new net V_D23: U$17.VO, X13-2.S
- new net V_K11: U$3.VO, X8-1.S
- new net V_K12: U$9.VO, X9-1.S
- new net V_K13: U$15.VO, X10-1.S
- new net V_K21: U$4.VO, X8-2.S
- new net V_K22: U$10.VO, X9-2.S
- new net V_K23: U$16.VO, X10-2.S
- new net V_OUT11: U$2.VO, X5-1.S
- new net V_OUT12: U$8.VO, X6-1.S
- new net V_OUT13: U$14.VO, X7-1.S
- new net V_OUT21: U$1.VO, X5-2.S
- new net V_OUT22: U$7.VO, X6-2.S
- new net V_OUT23: U$13.VO, X7-2.S
- net K11: now also U$3.IN; no longer Q1.G
- net K12: now also U$9.IN; no longer Q3.G
- net K13: now also U$15.IN; no longer Q5.G
- net K21: now also U$4.IN; no longer Q2.G
- net K22: now also U$10.IN; no longer Q4.G
- net K23: now also U$16.IN; no longer Q6.G
- net L1: now also U$1.OUT; no longer D2.C, Q2.D
- net L2: now also Q2.D, U$1.IN, U$5.IN; no longer D3.A, D4.C, Q3.S, Q4.D
- net L3: now also Q1.D, U$2.IN, U$6.IN; no longer D5.A, D6.C, Q5.S, Q6.D
- net V+: now also U$1.V+, U$10.V+, U$11.V+, U$12.V+, U$13.V+, U$14.V+, U$15.V+, U$16.V+, U$17.V+, U$18.V+, U$2.V+, U$3.V+, U$4.V+, U$5.V+, U$6.V+, U$7.V+, U$8.V+, U$9.V+; no longer D1.C, D3.C, D5.C, Q1.D, Q3.D, Q5.D, X1-1.S
- net V-: now also U$1.V-, U$10.V-, U$11.V-, U$12.V-, U$13.V-, U$14.V-, U$15.V-, U$16.V-, U$17.V-, U$18.V-, U$2.V-, U$3.V-, U$4.V-, U$5.V-, U$6.V-, U$7.V-, U$8.V-, U$9.V-; no longer D2.A, D4.A, D6.A, Q2.S, Q4.S, Q6.S, X1-2.S
Other:
- moved on the sheet: D1, D2, D3, D4, D5, D6, Q1, Q2, Q3, Q4, Q5, Q6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

Commit message: Płytka, falownik update
Parts:
- removed D1, D2, D3, D4, D5, D6: 1N4942, diode:1N4942
- removed U$1, U$10, U$11, U$12, U$13, U$14, U$15, U$16, U$17, U$18, U$2, U$3, U$4, U$5, U$6, U$7, U$8, U$9: CURRENT_MEAS_D_V02, current_meas:CURRENT_MEAS_D_V02
- removed X10, X8, X9: 87758-0216, con-molex:87758-0216
- added IC1, IC2, IC3, IC4, IC5, IC6, IC7, IC8, IC9: A1382UA, allegro:A1382UA
- added JP1, JP10, JP11, JP12, JP13, JP14, JP15, JP2, JP3, JP4, JP5, JP6, JP7, JP8, JP9: (no value), jumper:JP1E
- added X14: 87758-0216, con-molex:87758-0216
- Q1, Q2, Q3, Q4, Q5, Q6: value BSS101 -> VN88AF; device transistor-fet:BSS101 -> transistor-fet:VN88AF
Connections:
- removed net L4: D3.A, Q3.S, U$7.OUT
- removed net L5: Q4.D, U$11.IN, U$7.IN
- removed net L6: Q3.D, U$12.IN, U$8.IN
- removed net L7: D5.A, Q5.S, U$13.OUT
- removed net L8: Q6.D, U$13.IN, U$17.IN
- removed net L9: Q5.D, U$14.IN, U$18.IN
- removed net N$10: D5.C, U$18.OUT
- removed net N$9: D6.C, U$17.OUT
- removed net V+: U$1.V+, U$10.V+, U$11.V+, U$12.V+, U$13.V+, U$14.V+, U$15.V+, U$16.V+, U$17.V+, U$18.V+, U$2.V+, U$3.V+, U$4.V+, U$5.V+, U$6.V+, U$7.V+, U$8.V+, U$9.V+
- removed net V-: U$1.V-, U$10.V-, U$11.V-, U$12.V-, U$13.V-, U$14.V-, U$15.V-, U$16.V-, U$17.V-, U$18.V-, U$2.V-, U$3.V-, U$4.V-, U$5.V-, U$6.V-, U$7.V-, U$8.V-, U$9.V-
- removed net VCC1: Q3.G, U$9.OUT
- removed net VCC2: Q4.G, U$10.OUT
- removed net VCC3: Q5.G, U$15.OUT
- removed net VCC4: Q6.G, U$16.OUT
- removed net VCC5: Q1.G, U$3.OUT
- removed net VCC6: Q2.G, U$4.OUT
- removed net V_D11: U$6.VO, X11-1.S
- removed net V_D12: U$12.VO, X12-1.S
- removed net V_D13: U$18.VO, X13-1.S
- removed net V_D21: U$5.VO, X11-2.S
- removed net V_D22: U$11.VO, X12-2.S
- removed net V_D23: U$17.VO, X13-2.S
- removed net V_K11: U$3.VO, X8-1.S
- removed net V_K12: U$9.VO, X9-1.S
- removed net V_K13: U$15.VO, X10-1.S
- removed net V_K21: U$4.VO, X8-2.S
- removed net V_K22: U$10.VO, X9-2.S
- removed net V_K23: U$16.VO, X10-2.S
- new net BNC_1: JP1.1, JP2.1, X11-1.S
- new net BNC_2: JP3.1, JP4.1, X12-1.S
- new net BNC_3: JP5.1, JP6.1, X13-1.S
- new net BNC_4: JP10.1, JP11.1, JP12.1, X14-1.S
- new net BNC_5: JP13.1, JP14.1, JP15.1, X11-2.S
- new net BNC_6: JP7.1, X12-2.S
- new net BNC_7: JP8.1, X13-2.S
- new net BNC_8: JP9.1, X14-2.S
- new net N$12: IC5.GND, Q3.D
- new net N$14: IC4.GND, Q4.D
- new net N$15: IC4.VCC, IC6.VCC, Q3.S
- new net N$2: IC3.GND
- new net N$23: IC8.GND, Q5.D
- new net N$25: IC7.GND, Q6.D
- new net N$26: IC7.VCC, IC9.VCC, Q5.S
- new net N$3: IC1.GND, Q2.D
- net GND: no longer D2.A, D4.A, D6.A, U$1.GND, U$10.GND, U$11.GND, U$12.GND, U$13.GND, U$14.GND, U$15.GND, U$16.GND, U$17.GND, U$18.GND, U$2.GND, U$3.GND, U$4.GND, U$5.GND, U$6.GND, U$7.GND, U$8.GND, U$9.GND
- net K11: now also JP10.2, Q1.G; no longer U$3.IN
- net K12: now also JP11.2, Q3.G; no longer U$9.IN
- net K13: now also JP12.2, Q5.G; no longer U$15.IN
- net K21: now also JP13.2, Q2.G; no longer U$4.IN
- net K22: now also JP14.2, Q4.G; no longer U$10.IN
- net K23: now also JP15.2, Q6.G; no longer U$16.IN
- net L1: now also IC3.OUT, JP9.2; no longer D1.A, Q1.S, U$1.OUT
- net L2: now also IC6.OUT, JP8.2; no longer Q2.D, U$1.IN, U$5.IN
- net L3: now also IC9.OUT, JP7.2; no longer Q1.D, U$2.IN, U$6.IN
- net N$1: now also IC2.GND, Q1.D; no longer D1.C, U$6.OUT
- net N$4: now also IC1.VCC, IC3.VCC, Q1.S; no longer D4.C, U$11.OUT
- net N$5: now also IC6.GND; no longer D2.C, U$5.OUT
- net N$6: now also IC9.GND; no longer D3.C, U$12.OUT
- net VCC: now also IC2.VCC, IC5.VCC, IC8.VCC; no longer U$14.OUT, U$2.OUT, U$8.OUT
- net V_OUT11: now also IC2.OUT, JP1.2; no longer U$2.VO
- net V_OUT12: now also IC5.OUT, JP3.2; no longer U$8.VO
- net V_OUT13: now also IC8.OUT, JP5.2; no longer U$14.VO
- net V_OUT21: now also IC1.OUT, JP2.2; no longer U$1.VO
- net V_OUT22: now also IC4.OUT, JP4.2; no longer U$7.VO
- net V_OUT23: now also IC7.OUT, JP6.2; no longer U$13.VO
Other:
- moved on the sheet: Q1, Q2, Q3, Q4, Q5, Q6, X1-1, X1-2, X11-1, X11-2, X12-1, X12-2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
