File: Schematy eagle/Falownik/falownik.sch (EAGLE design)
At the start: 41 parts, among them IC1 A1382UA, IC2 A1382UA, IC3 A1382UA, IC4 A1382UA, IC5 A1382UA, IC6 A1382UA, IC7 A1382UA, IC8 A1382UA, IC9 A1382UA, Q1 VN88AF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

Commit message: dodanie pinow kodujacych zadanie
Parts:
- added JP16: (no value), jumper:JP1E
- added R1: 1k, eagle-ltspice:R0204/7
- added X10, X8, X9: 87758-0216, con-molex:87758-0216
Connections:
- new net 0: X10-1.S
- new net CODE: JP16.2, R1.1, X8-1.S, X8-2.S, X9-1.S, X9-2.S
- new net CODE_1F/3F: JP16.1, X10-2.S
- net VCC: now also R1.2
Other:
- moved on the sheet: X11-1, X11-2, X12-1, X12-2, X13-1, X13-2, X14-1, X14-2
