File: Schematy eagle/Płytka/layout.sch (EAGLE design)
At the start: 2 parts

Commit message: Update
Parts:
- added J1, J10, J11, J12, J2, J3, J4, J5, J6: (no value), SparkFun-Connectors:BANANA_CONN
Connections:
- new net GND: J10.1, J11.1, J12.1
- new net L1: J1.1
- new net L2: J2.1
- new net L3: J3.1
- new net V+: J4.1, J5.1, J6.1

Commit message: Płytka, falownik update
Parts:
- removed J1, J2, J3: (no value), SparkFun-Connectors:BANANA_CONN
- added U$1: STM32F40XSTM32D40X, stm32f:STM32F40XSTM32D40X
- added X1, X2, X3, X4, X5, X6, X7, X8: BN35N61, con-coax:BN35N61
Connections:
- removed net L1: J1.1
- removed net L2: J2.1
- removed net L3: J3.1
- new net N$10: SV2.37, X5.1
- new net N$11: SV2.27, X6.1
- new net N$12: SV2.3, X8.1
- new net N$13: SV2.11, X7.1
- new net N$2: SV1.39
- new net N$3: SV1.33
- new net N$4: SV1.40
- new net N$5: SV1.34
- new net N$6: SV2.2, X1.1
- new net N$7: SV2.10, X2.1
- new net N$8: SV2.30, X3.1
- new net N$9: SV2.40, X4.1
- net GND: now also X1.2, X2.2, X4.2, X6.2, X7.2, X8.2

Commit message: Update płytka, falownik
Parts:
- removed SV1, SV2: (no value), con-lstb:MA20-2
- removed U$1: STM32F40XSTM32D40X, stm32f:STM32F40XSTM32D40X
- removed X1, X2, X3, X4, X5, X6, X7, X8: BN35N61, con-coax:BN35N61
- added J1, J2: ZIFSOCKET-28-3", SparkFun-Connectors:ZIFSOCKET-28-3"
- added U$2: STM32F40XSTM32D40X, stm32f:STM32F40XSTM32D40X
- added X10, X11, X12, X13, X14, X15, X16, X9: BN35N61, con-coax:BN35N61
Connections:
- removed net N$10: SV2.37, X5.1
- removed net N$11: SV2.27, X6.1
- removed net N$12: SV2.3, X8.1
- removed net N$13: SV2.11, X7.1
- removed net N$2: SV1.39
- removed net N$3: SV1.33
- removed net N$4: SV1.40
- removed net N$5: SV1.34
- removed net N$6: SV2.2, X1.1
- removed net N$7: SV2.10, X2.1
- removed net N$8: SV2.30, X3.1
- removed net N$9: SV2.40, X4.1
- new net BNC_1: J2.P$1
- new net BNC_2: J2.P$5, X10.1
- new net BNC_3: J2.P$10, X11.1
- new net BNC_4: J2.P$14, X12.1
- new net BNC_5: J2.P$15, X13.1
- new net BNC_6: J2.P$19, X14.1
- new net BNC_7: J2.P$24, X15.1
- new net BNC_8: J2.P$28, X16.1
- net GND: now also X10.2, X11.2, X12.2, X13.2, X14.2, X15.2, X16.2, X9.2; no longer X1.2, X2.2, X4.2, X6.2, X7.2, X8.2
